File: hardware/kicad/QRPTransceiver.kicad_pcb (KiCad board)
At the start: 2 copper layers, 162.5 x 99 mm, 252 parts, among them J1 Data, J2 Power, J3 Input, J5 Audio Gain, J6 Audio Out, J7 Speaker, Q1 VN10N, Q2 2SK2394, Q3 2SK2394, Q4 J177, Q5 2N3904, Q6 2N3904, Q7 VN10LF, Q8 VN10LF, T1 Input, U1 AP1117-50, U10 LM386, U2 Si5351Module, U3 FST3253, U4 TS924, U5 TS924, U6 OPA1641, U7 TS924, U8 TS924, U9 OPA1641

Commit message: Firmware: encoder ISR queue, S-meter calibration, UI polish, SI5351 fixes
Firmware changes:
- RotaryInput: rewrite to interrupt-driven ISR queue (RP2040 GPIO callback,
  64-event ring buffer). Eliminates ~2-3 step/sec polling limit.
- SI5351Control: add liveRetune param to setQuadrature90(). Live-retune path
  skips PLL reset and output disable/enable to eliminate audio transients.
  Both CLK0/CLK1 forced to PLLA for phase coherence. Phase registers zeroed
  in all low-band paths.
- BoardControl: S-meter ADC inversion (higher V = weaker signal), configurable
  zero-raw floor, gain permille, and optional sqrt log companding.
- main.cpp: analogReadResolution(12) for 12-bit ADC. S_METER_ZERO_RAW=372
  (~3V floor), GAIN=1220, LOG=true. Tune coalescing via flushPendingTuneDelta.
  40ms display refresh throttle. S-meter suppressed during tuning (120ms).
  LED steady on (no heartbeat). SI5351 correction -4610000 PPB.
- DisplayUI: step indicator label, flashTuneDirection (UP/DN), step digit
  flash with 500ms duration on encoder button press.
- upload_uf2.py: wait-for-mount loop + picotool fallback upload.

Hardware:
- KiCAD PCB and schematic updates (mixer sheet, audio sheet)
Parts:
- added C24: 100n, Capacitor_SMD:C_0805_2012Metric, F.Cu at (171.6, 29.0)
- added C25: 100n, Capacitor_SMD:C_0805_2012Metric, F.Cu at (171.6, 32.0)
- added C76: 100n, Capacitor_SMD:C_0805_2012Metric, F.Cu at (162.8, 33.8)
- C92: footprint Capacitor_SMD:CP_Elec_3x5.3 -> Capacitor_SMD:CP_Elec_6.3x4.9
- D3, D4: footprint Diode_SMD:D_0805_2012Metric -> Diode_SMD:D_1206_3216Metric
- D5: footprint Inductor_SMD:L_0805_2012Metric -> Diode_SMD:D_1206_3216Metric
- moved C92 1.64 mm to (147.8, 73.5)
- moved C83 1.50 mm to (147.1, 68.5)
Routing:
- net GND: track 185.2 -> 187.1 mm
- net /Sheet6280C94B/AudioAGC: track 25.6 -> 23.8 mm
- net Net-(C92-Pad1): track 9.41 -> 8.17 mm
- net CWMUTE: track 64.1 -> 64.6 mm
