File: hardware/kicad/FrontendMixer.kicad_sch (KiCad schematic)
At the start: 75 parts, among them J11 Exciter Out, J3 Receive Input, Q10 J310, Q11 2N3904, Q2 2N3904, Q9 J310, T1 Transformer_1P_1S, T2 Transformer_1P_2S, T3 Transformer_1P_1S, U2 Si5351Module, U3 FST3253, U9 FST3253

Commit message: Document SSC notes reference in CURRENT_SI5351_APPROACH.md
Parts:
- renumbered C95 to C10, C114 to C11, C115 to C12, C93 to C13, C87 to C14, C12 to C15, C83 to C16, C85 to C17, C13 to C18, C14 to C19, C110 to C2, C92 to C20, C15 to C21, C16 to C22, C17 to C23, C148 to C24, C150 to C25, C18 to C26, C147 to C27, C149 to C28, C118 to C3, C111 to C4, C117 to C5, C11 to C6, C112 to C7, C113 to C8, C116 to C9, J3 to J1, J11 to J2, L4 to L1, L5 to L2, Q2 to Q1, Q9 to Q2, Q10 to Q3, Q11 to Q4, R114 to R1, R133 to R10, R132 to R11, R131 to R12, R120 to R13, R121 to R14, R122 to R15, R85 to R16, R11 to R17, R89 to R18, R12 to R19, R136 to R2, R13 to R20, R78 to R21, R80 to R22, R81 to R23, R82 to R24, R91 to R25, R94 to R26, R95 to R27, R127 to R28, R126 to R29, R115 to R3, R128 to R30, R129 to R31, R130 to R32, R116 to R4, R117 to R5, R135 to R6, R118 to R7, R134 to R8, R119 to R9, RV2 to RV1, T3 to T1, T1 to T3, U2 to U1, U3 to U2, U9 to U3
