File: hardware/kicad/exciterAudio.kicad_sch (KiCad schematic)
At the start: 79 parts, among them J12 Mic, U13 LM324, U14 LM324, U15 TS924

Commit message: Document SSC notes reference in CURRENT_SI5351_APPROACH.md
Parts:
- removed J12: Mic, symbol Connector:Conn_01x02_Socket
- removed U13: LM324, symbol Amplifier_Operational:LM324
- removed unit 5 of U14
- added J20: Mic, symbol Connector_Generic:Conn_01x02
- renumbered C153 to C123, C151 to C124, C155 to C125, C154 to C126, C152 to C127, C119 to C128, C120 to C129, C121 to C130, C122 to C131, C123 to C132, C124 to C133, C125 to C134, C126 to C135, C127 to C136, C128 to C137, C129 to C138, C130 to C139, C131 to C140, C132 to C141, C133 to C142, C134 to C143, C135 to C144, C136 to C145, C137 to C146, C138 to C147, C139 to C148, C140 to C149, C141 to C150, C142 to C151, C143 to C152, C144 to C153, C145 to C154, C146 to C155, R167 to R137, R168 to R138, R169 to R139, R166 to R140, R170 to R141, R165 to R142, R171 to R143, R177 to R144, R176 to R145, R172 to R146, R174 to R147, R173 to R148, R175 to R149, R137 to R150, R138 to R151, R139 to R152, R140 to R153, R141 to R154, R142 to R155, R143 to R156, R144 to R157, R145 to R158, R146 to R159, R147 to R160, R148 to R161, R149 to R162, R150 to R163, R151 to R164, R152 to R165, R153 to R166, R154 to R167, R155 to R168, R156 to R169, R157 to R170, R158 to R171, R159 to R172, R160 to R173, R161 to R174, R162 to R175, R163 to R176, R164 to R177
Connections:
- net GND: now also J20.1 (Pin_1)
- net at RV3.1: now also J20.2 (Pin_2)
- net +12V: now reaches R142.1
