File: hardware/kicad/receivePolyphase.kicad_sch (KiCad schematic)
At the start: 93 parts, among them U4 TS924, U5 TS924, U6 OPA1641

Commit message: Document SSC notes reference in CURRENT_SI5351_APPROACH.md
Parts:
- renumbered C20 to C29, C21 to C30, C22 to C31, C23 to C32, C28 to C33, C29 to C34, C30 to C35, C31 to C36, C32 to C37, C33 to C38, C34 to C39, C35 to C40, C36 to C41, C37 to C42, C38 to C43, C39 to C44, C40 to C45, C41 to C46, C42 to C47, C43 to C48, C44 to C49, C45 to C50, C46 to C51, C47 to C52, C48 to C53, C49 to C54, C50 to C55, C51 to C56, C52 to C57, C53 to C58, C54 to C59, C55 to C60, C56 to C61, C57 to C62, C58 to C63, C59 to C64, C60 to C65, C61 to C66, C62 to C67, C63 to C68, C64 to C69, R14 to R33, R15 to R34, R16 to R35, R17 to R36, R18 to R37, R19 to R38, R20 to R39, R21 to R40, R22 to R41, R23 to R42, R24 to R43, R25 to R44, R26 to R45, R27 to R46, R28 to R47, R29 to R48, R30 to R49, R31 to R50, R32 to R51, R33 to R52, R34 to R53, R35 to R54, R36 to R55, R37 to R56, R38 to R57, R39 to R58, R40 to R59, R41 to R60, R42 to R61, R43 to R62, R44 to R63, R45 to R64, R46 to R65, R47 to R66, R48 to R67, R49 to R68, R50 to R69, R51 to R70, R52 to R71, R53 to R72, R54 to R73, R55 to R74, R56 to R75, R57 to R76, R58 to R77, R59 to R78, R60 to R79, R61 to R80, R62 to R81
Other:
- moved on the sheet: C29, C30, C31, C32, C33, C34, C35, C36, C37, C38, C39, C40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
