File: hardware/kicad/controller/POWER_CIRCUIT_CONTROLLER_SHEET.kicad_sch (KiCad schematic)
At the start: 1 part

Commit message: Simplify kicad sheet: remove title_block to avoid comment parsing issues
Other:
- company: QRPTransceiver -> (none)
- title: Controller: Processor Power Latch -> (none)
Changed lines of the file:
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@@
 (kicad_sch (version 20211014) (generator eeschema)
-  (paper "A4")
-  (title_block
-    (title "Controller: Processor Power Latch")
-    (company "QRPTransceiver")
-    (rev "0.1")
-    (date "2026-08-29")
-    (comment "Draft schematic sheet for the processor power-latch. Update symbols/footprints in KiCad.")
-  )
-  ;; Minimal valid symbol entries (generic). Replace with real library parts in KiCad.
+  ;; Minimal sheet without title_block to avoid parser issues.
+  ;; Replace generic symbols with real library parts inside KiCad.
   (symbol (lib_id "Device:R") (at 50 40 0) (unit 1) (value "R1") (footprint "Resistor_SMD:R_0603_1608Metric") (property "Value" "1M"))
   (symbol (lib_id "Device:R") (at 50 80 0) (unit 1) (value "R2") (footprint "Resistor_SMD:R_0603_1608Metric") (property "Value" "1k"))
@@
   (wire (pts (xy 200 100) (xy 200 140)))
   (label (name "POWER_HOLD") (at 210 120 0) (orientation 0))
-  (comment "Note: Update library links and footprints in KiCad.")
 )
