File: hardware/kicad/controller/POWER_CIRCUIT_CONTROLLER_SHEET.kicad_sch (KiCad schematic)
At the start: 1 part

Commit message: Consolidate controller power sheet to single KiCad-8 compatible schematic
Parts:
- ?: value 100nF -> LDO_3V3; symbol Device:C -> Regulator:LD
Changed lines of the file:
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@@
 (kicad_sch (version 20220628) (generator eeschema)
+  (paper "A4")
+  ;; Consolidated minimal KiCad 8 schematic sheet for controller power-latch.
+  ;; Import into KiCad and replace the generic symbols with your project libraries.
   (symbol (lib_id "Device:R") (at 50 40 0) (unit 1) (value "R1") (footprint "Resistor_SMD:R_0603_1608Metric") (property "Value" "1M"))
   (symbol (lib_id "Device:R") (at 50 80 0) (unit 1) (value "R2") (footprint "Resistor_SMD:R_0603_1608Metric") (property "Value" "1k"))
-  (symbol (lib_id "Device:C") (at 140 40 0) (unit 1) (value "C1") (footprint "Capacitor_SMD:C_0603_1608Metric") (property "Value" "100nF"))
-  (wire (pts (xy 20 60) (xy 60 60)))
-  (wire (pts (xy 60 60) (xy 120 60)))
-  (wire (pts (xy 120 60) (xy 160 60)))
-)
-(kicad_sch (version 20211014) (generator eeschema)
-  (symbol (lib_id "Device:R") (at 50 40 0) (unit 1) (value "R1") (footprint "Resistor_SMD:R_0603_1608Metric") (property "Value" "1M"))
-  (symbol (lib_id "Device:R") (at 50 80 0) (unit 1) (value "R2") (footprint "Resistor_SMD:R_0603_1608Metric") (property "Value" "1k"))
-  (symbol (lib_id "Device:C") (at 140 40 0) (unit 1) (value "C1") (footprint "Capacitor_SMD:C_0603_1608Metric") (property "Value" "100nF"))
-  (wire (pts (xy 20 60) (xy 60 60)))
-  (label (name "VIN") (at 5 60 0) (orientation 180))
-  (wire (pts (xy 60 60) (xy 120 60)))
-  (label (name "GATE_CTRL") (at 95 75 0) (orientation 0))
-  (wire (pts (xy 120 60) (xy 160 60)))
-  (label (name "V_SYS") (at 170 60 0) (orientation 0))
-)
- (kicad_sch (version 20211014) (generator eeschema)
-  (paper "A4")
-  ;; Minimal valid sheet content. Import into KiCad and replace symbols/footprints
-  ;; with the project's libraries.
-  (symbol (lib_id "Device:R") (at 50 40 0) (unit 1) (value "R1") (footprint "Resistor_SMD:R_0603_1608Metric") (property "Value" "1M"))
-  (symbol (lib_id "Device:R") (at 50 80 0) (unit 1) (value "R2") (footprint "Resistor_SMD:R_0603_1608Metric") (property "Value" "1k"))
