File: hardware/kicad/controller/POWER_CIRCUIT_CONTROLLER_SHEET.kicad_sch (KiCad schematic)
At the start: 1 part

Commit message: Temporary: remove symbols to avoid lib_id parsing error; minimal sheet
Parts:
- removed ?: LDO_3V3, symbol Regulator:LD
Changed lines of the file:
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@@
 (kicad_sch (version 20220628) (generator eeschema)
+  (paper "A4")
+  (wire (pts (xy 20 60) (xy 60 60)))
+  (label (name "VIN") (at 5 60 0) (orientation 180))
+  (wire (pts (xy 60 60) (xy 120 60)))
+  (label (name "GATE_CTRL") (at 95 75 0) (orientation 0))
+  (wire (pts (xy 120 60) (xy 160 60)))
+  (label (name "V_SYS") (at 170 60 0) (orientation 0))
+  (wire (pts (xy 140 120) (xy 140 80)))
+  (label (name "GND") (at 140 150 0) (orientation 0))
+  (wire (pts (xy 200 100) (xy 200 140)))
+  (label (name "POWER_HOLD") (at 210 120 0) (orientation 0))
+)
+ (kicad_sch (version 20220628) (generator eeschema)
   (symbol (lib_id "Device:R") (at 50 40 0) (unit 1) (value "R1") (footprint "Resistor_SMD:R_0603_1608Metric") (property "Value" "1M"))
   (symbol (lib_id "Device:R") (at 50 80 0) (unit 1) (value "R2") (footprint "Resistor_SMD:R_0603_1608Metric") (property "Value" "1k"))

Commit message: Add placeholder symbol to satisfy KiCad parser
Parts:
- added ?: (no value), symbol Device:R
Changed lines of the file:
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@@
 (kicad_sch (version 20220628) (generator eeschema)
-  (paper "A4")
+  (symbol (lib_id "Device:R") (at 50 40 0) (unit 1) (value "R1"))
   (wire (pts (xy 20 60) (xy 60 60)))
   (label (name "VIN") (at 5 60 0) (orientation 180))
