File: hardware/kicad/controller/controller.kicad_sch (KiCad schematic)
At the start: 42 parts, among them J10 Filter Board, J11 Power Amp, J12 Power on/off, J13 Function2, J14 Function 1, J15 Band, J16 Mode, J17 Rotary Encoder, J18 Display, J19 Power, U12 AP1117-50, U13 LM324, U14 LM324, U4 TS924, U5 TS924, U7 TS924, U8 TS924

Commit message: Save local KiCad edits
Connections:
- net TXRX: no longer J11.3 (Pin_3)
Other:
- moved on the sheet: A1, R178, R179
